File: esp32_radio.kicad_pcb (KiCad board)
At the start: 2 copper layers, 76.2 x 73.7 mm, 130 parts, among them J1 RP-SMA, J3 Conn_ADC, U1 ILI9341_TOUCH_SD, U2 RF4IN1, U3 esp32-lolin32, U4 WS2812B, U5 Joystick, U6 Joystick, U7 MCP3008, U8 MAX98357a, U9 nRF24L01

Commit message: v4
Parts:
- removed REF** (x108): Via, spectre:Via
- added BT1: Battery_Cell, Connectors_JST:JST_PH_S2B-PH-SM4-TB_02x2.00mm_Angled, F.Cu at (128.2, 109.1)
- added BZ1: Buzzer, Buzzers_Beepers:Buzzer_12x9.5RM7.6, B.Cu at (111.2, 80.1)
- added C10: 220pF, Capacitors_SMD:C_0805, F.Cu at (37.1, 49.0)
- added C11: 0.1µF, Capacitors_SMD:C_0805, B.Cu at (266.2, 102.9)
- added C12: 10µF, Capacitors_SMD:C_0805, B.Cu at (266.2, 104.9)
- added C13: ???, Capacitors_SMD:C_0805, F.Cu at (142.2, 86.1)
- added C14: 10uF, Capacitors_SMD:C_0805, F.Cu at (143.2, 112.1)
- added C8: 220pF, Capacitors_SMD:C_0805, F.Cu at (32.5, 47.0)
- added C9: 0.1uF, Capacitors_SMD:C_0805, F.Cu at (38.1, 43.2)
- added D1: MBR120, Diodes_SMD:D_SOD-123, F.Cu at (113.2, 91.1)
- added D2: orange, LEDs:LED_0805, F.Cu at (116.2, 99.1)
- added J2: LCD_TS, spectre:TFT-2.4-IlI9341-18pin, B.Cu at (179.9, 91.6)
- added J4: USB_OTG, Connectors_USB:USB_Micro-B_Wuerth-629105150521, F.Cu at (117.9, 110.3)
- added J5: Micro_SD_Card, Connectors:microSD_Card_Receptacle_Wuerth_693072010801, F.Cu at (180.2, 79.6)
- added J6: GS2, Connectors:GS2, F.Cu at (42.9, 188.3)
- added J7: Conn_ADC, Pin_Headers:Pin_Header_Straight_2x04_Pitch2.54mm, F.Cu at (265.7, 90.7)
- added Q1: DMG3415U, TO_SOT_Packages_SMD:SOT-23, F.Cu at (117.2, 94.1)
- added Q2: Q_NPN_BCE, TO_SOT_Packages_SMD:SOT-23, F.Cu at (155.2, 111.1)
- added Q3: Q_NPN_BCE, TO_SOT_Packages_SMD:SOT-23, F.Cu at (155.2, 106.1)
- added Q4: Q_NPN_BCE, TO_SOT_Packages_SMD:SOT-23, F.Cu at (111.2, 76.1)
- added R10: 10K, Resistors_SMD:R_0805, F.Cu at (169.4, 83.1)
- added R11: 10K, Resistors_SMD:R_0805, F.Cu at (169.5, 81.1)
- added R12: 10K, Resistors_SMD:R_0805, F.Cu at (169.5, 79.0)
- added R13: 100K, Resistors_SMD:R_0805, F.Cu at (47.8, 189.5)
- added R14: 100K, Resistors_SMD:R_0805, F.Cu at (36.1, 188.2)
- added R2: 100K, Resistors_SMD:R_0805, F.Cu at (121.2, 94.1)
- added R3: 1k, Resistors_SMD:R_0805, F.Cu at (120.2, 99.1)
- added R4: 10K, Resistors_SMD:R_0805, F.Cu at (150.1, 110.1)
- added R5: 10K, Resistors_SMD:R_0805, F.Cu at (150.2, 106.1)
- added R6: 4.7K, Resistors_SMD:R_0805, F.Cu at (129.2, 100.1)
- added R7: 3.9R, Resistors_SMD:R_0805, F.Cu at (60.7, 142.8)
- added R8: 4.7R, Resistors_SMD:R_0805, F.Cu at (112.2, 85.1)
- added R9: 1M, Resistors_SMD:R_0805, F.Cu at (27.7, 42.9)
- added U10: MCP3008, Housings_SOIC:SOIC-16_3.9x9.9mm_Pitch1.27mm, B.Cu at (269.6, 97.4)
- added U11: Joystick, spectre:Joystick_raider, B.Cu at (177.2, 51.6)
- added U12: Joystick, spectre:Joystick_raider, B.Cu at (117.2, 51.6)
- C1: value 1µF -> 10uF
- C3: value 0.1uF -> 1uF
- C4: value 0.1µF -> 10uF; moved to F.Cu
- C5: value 10µF -> 10uF; moved to F.Cu
- C6: value 220pF -> 1µF; moved to B.Cu
- C7: value 220pF -> 10uF
- J1: footprint tinkerforge:CON-SMA-EDGE -> spectre:CON-SMA-EDGE; moved to F.Cu
- J3: value Conn_ADC -> GS2; footprint Pin_Headers:Pin_Header_Straight_2x04_Pitch2.54mm -> Connectors:GS2
- R1: value 1M -> 100k
- U1: value ILI9341_TOUCH_SD -> RF4IN1; footprint spectre:LCD -> spectre:RF4IN1
- U2: value RF4IN1 -> AP2112-3.3; footprint spectre:RF4IN1 -> TO_SOT_Packages_SMD:SOT-23-5; moved to F.Cu
- U3: value esp32-lolin32 -> ESP32-WROOM; footprint spectre:esp32-lolin32 -> spectre:ESP32-WROOM; moved to F.Cu
- U4: value WS2812B -> nRF24L01; footprint LEDs:LED_WS2812B-PLCC4 -> RF_Modules:nRF24L01_Breakout
- U5: value Joystick -> MCP73831; footprint spectre:Joystick_raider -> TO_SOT_Packages_SMD:TSOT-23-5
- U6: value Joystick -> WS2812B; footprint spectre:Joystick_raider -> LEDs:LED_WS2812B-PLCC4; moved to B.Cu
- U7: value MCP3008 -> MAX98357a; footprint Housings_SOIC:SOIC-16_3.9x9.9mm_Pitch1.27mm -> Housings_DFN_QFN:QFN-16-1EP_3x3mm_Pitch0.5mm; moved to F.Cu
- U8: value MAX98357a -> CP2104; footprint Housings_DFN_QFN:QFN-16-1EP_3x3mm_Pitch0.5mm -> Housings_DFN_QFN:QFN-24-1EP_4x4mm_Pitch0.5mm
- U9: value nRF24L01 -> XPT2046TS; footprint RF_Modules:nRF24L01_Breakout -> Housings_SSOP:TSSOP-16_4.4x5mm_Pitch0.65mm; moved to F.Cu
- moved C7 138.5 mm to (32.8, 42.7), turned to 0 degrees
- moved U7 127.7 mm to (50.5, 43.0), turned to 0 degrees
- moved L2 116.4 mm to (51.9, 52.6), turned to 0 degrees
- moved L1 111.8 mm to (57.5, 48.3), turned to 0 degrees
- moved LS1 107.3 mm to (68.1, 50.0)
- moved U1 68.1 mm to (147.7, 59.6)
- moved J3 56.1 mm to (116.8, 85.1)
- moved C6 54.2 mm to (139.7, 56.6), turned to 90 degrees
- moved C5 52.6 mm to (120.2, 103.1)
- moved U5 47.2 mm to (124.9, 100.0)
- moved C1 39.2 mm to (120.2, 90.1), turned to 180 degrees
- moved U2 35.3 mm to (125.2, 91.1), turned to 0 degrees
- moved C4 35.1 mm to (135.2, 91.1), turned to 270 degrees
- moved R1 34.4 mm to (113.2, 95.1)
- moved U6 29.5 mm to (147.2, 56.6), turned to 0 degrees
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Connections:
- C1 pad 1: +3V3 -> Net-(C1-Pad1)
- C2 pad 1: +5V -> +3V3
- C3 pad 1: +5V -> +3V3
- C5 pad 1: +3V3 -> VBAT
- C6 pad 1: Net-(C6-Pad1) -> +3V3
- C7 pad 1: Net-(C7-Pad1) -> +5V
- J3 pad 1: /EXT_ADC_CH0 -> Net-(J3-Pad1)
- J3 pad 2: /EXT_ADC_CH1 -> /I2S_DATA
- L1 pad 1: Net-(C7-Pad1) -> Net-(C10-Pad1)
- L2 pad 1: Net-(C6-Pad1) -> Net-(C8-Pad1)
- LS1 pad 1: Net-(C7-Pad1) -> Net-(C10-Pad1)
- LS1 pad 2: Net-(C6-Pad1) -> Net-(C8-Pad1)
- R1 pad 1: Net-(R1-Pad1) -> VBUS
- R1 pad 2: +5V -> GND
- U1 pad 1: Net-(U1-Pad1) -> +3V3
- U1 pad 10: /LCD_CMD -> /MOSI
- U1 pad 11: +3V3 -> /MISO
- U1 pad 12: /CS_LCD -> /CYRF_RST
- U1 pad 14: +3V3 -> GND
- U1 pad 15: /SCK -> GND
- U1 pad 16: /MISO -> Net-(J1-Pad1)
- U1 pad 17: /MOSI -> GND
- U1 pad 18: /CS_SD -> GND
- U1 pad 2: /MISO -> GND
- U1 pad 3: /MOSI -> /PE1
- U1 pad 4: /CS_TOUCH -> /PE2
- U1 pad 5: /SCK -> /CS_A7105
- U1 pad 6: /MISO -> /CS_CC25
- U1 pad 7: +3V3 -> /CS_NRF24
- U1 pad 8: /SCK -> /CS_CYRF
- U1 pad 9: /MOSI -> /SCK
- U2 pad 1: +3V3 -> Net-(C1-Pad1)
- U2 pad 3: /PE1 -> Net-(R2-Pad2)
- U2 pad 4: /PE2 -> Net-(U2-Pad4)
- U2 pad 5: /CS_A7105 -> +3V3
- U3 pad 1: +3V3 -> GND
- U3 pad 10: /I2S_BCLK -> /I2S_LRC
- U3 pad 11: /CS_CC25 -> /I2S_BCLK
- U3 pad 12: /CS_A7105 -> /CS_CC25
- U3 pad 13: /PE2 -> /CS_A7105
- U3 pad 14: /PE1 -> /PE2
- U3 pad 15: +5V -> GND
- U3 pad 16: GND -> /PE1
- U3 pad 17: /CS_LCD -> Net-(U3-Pad17)
- U3 pad 18: /LCD_CMD -> Net-(U3-Pad18)
- U3 pad 19: GND -> Net-(U3-Pad19)
- U3 pad 2: Net-(U3-Pad2) -> +3V3
- U3 pad 21: /CS_TOUCH -> Net-(U3-Pad21)
- U3 pad 22: /CS_SD -> Net-(U3-Pad22)
- U3 pad 23: /CYRF_RST -> /CS_LCD
- U3 pad 24: +3V3 -> /LCD_CMD
- U3 pad 25: /NEOPIXEL -> /GPIO_0
- U3 pad 26: /SCK -> /CS_TOUCH
- U3 pad 27: /MOSI -> /CS_SD
- U3 pad 28: /MISO -> /CYRF_RST
- U3 pad 29: GND -> /NEOPIXEL
- U3 pad 3: /INT_ADC_CH0 -> /RESET
- U3 pad 30: GND -> /SCK
- U3 pad 31: /CS_ADC -> /MISO
- U3 pad 32: /I2S_DATA -> Net-(U3-Pad32)
- U3 pad 33: +3V3 -> /CS_ADC
- U3 pad 36: GND -> /I2S_DATA
- U3 pad 4: /INT_ADC_CH1 -> /INT_ADC_CH0
- U3 pad 5: /CS_CYRF -> /INT_ADC_CH1
- U3 pad 6: /CS_NRF24 -> /INT_ADC_CH2
- U3 pad 7: /INT_ADC_CH2 -> /INT_ADC_CH3
- U3 pad 8: /INT_ADC_CH3 -> /CS_CYRF
- U3 pad 9: /I2S_LRC -> /CS_NRF24
- U4 pad 1: +3V3 -> GND
- U4 pad 2: Net-(U4-Pad2) -> +3V3
- U4 pad 3: GND -> +3V3
- U4 pad 4: /NEOPIXEL -> /CS_NRF24
- U5 pad 5: +3V3 -> Net-(R6-Pad2)
- U7 pad 1: /EXT_ADC_CH0 -> /I2S_DATA
- U7 pad 10: /CS_ADC -> Net-(L1-Pad2)
- U7 pad 11: /MOSI -> GND
- U7 pad 12: /MISO -> Net-(U7-Pad12)
- U7 pad 13: /SCK -> Net-(U7-Pad13)
- U7 pad 14: GND -> /I2S_LRC
- U7 pad 15: +3V3 -> GND
- U7 pad 16: +3V3 -> /I2S_BCLK
- U7 pad 2: /EXT_ADC_CH1 -> Net-(U7-Pad2)
- U7 pad 3: /EXT_ADC_CH2 -> GND
- U7 pad 4: /EXT_ADC_CH3 -> Net-(R9-Pad1)
- U7 pad 5: /EXT_ADC_CH4 -> Net-(U7-Pad5)
- U7 pad 6: /EXT_ADC_CH5 -> Net-(U7-Pad6)
- U7 pad 7: /EXT_ADC_CH6 -> +5V
- U7 pad 8: /EXT_ADC_CH7 -> +5V
- U7 pad 9: GND -> Net-(L2-Pad2)
- U8 pad 1: /I2S_DATA -> Net-(U8-Pad1)
- U8 pad 10: Net-(L1-Pad2) -> Net-(U8-Pad10)
- U8 pad 11: GND -> Net-(U8-Pad11)
- U8 pad 14: /I2S_LRC -> Net-(U8-Pad14)
- U8 pad 15: GND -> Net-(U8-Pad15)
- U8 pad 16: /I2S_BCLK -> Net-(U8-Pad16)
- U8 pad 17: (no net) -> Net-(U8-Pad17)
- U8 pad 2: Net-(U8-Pad2) -> GND
- U8 pad 3: GND -> /D-
- U8 pad 4: Net-(R1-Pad1) -> /D+
- U8 pad 5: Net-(U8-Pad5) -> +3V3
- U8 pad 6: Net-(U8-Pad6) -> +3V3
- U8 pad 7: +5V -> +3V3
- U8 pad 8: +5V -> VBUS
- U8 pad 9: Net-(L2-Pad2) -> Net-(U8-Pad9)
- U9 pad 1: GND -> +3V3
- U9 pad 2: +3V3 -> /TS_X+
- U9 pad 3: +3V3 -> /TS_Y+
- U9 pad 4: /CS_NRF24 -> /TS_X-
- U9 pad 5: /SCK -> /TS_Y-
- U9 pad 6: /MOSI -> GND
- U9 pad 7: /MISO -> VBAT
Routing:
- net +3V3: track 262.4 -> 26.2 mm, vias 3 -> 0
- net /MISO: track 169.6 -> 0.00 mm, vias 5 -> 0
- net /MOSI: track 161.5 -> 0.00 mm, vias 8 -> 0
- net /SCK: track 144.4 -> 0.00 mm, vias 2 -> 0
- net /NEOPIXEL: track 73.9 -> 0.00 mm, vias 5 -> 0
- net /CS_SD: track 69.6 -> 0.00 mm, vias 2 -> 0
- net /CS_ADC: track 63.5 -> 0.00 mm, vias 2 -> 0
- net /EXT_ADC_CH1: track 61.1 -> 0.00 mm
- net VBUS: track 0.00 -> 56.6 mm, vias 0 -> 2
- net /CYRF_RST: track 55.8 -> 0.00 mm, vias 4 -> 0
- net /EXT_ADC_CH0: track 54.4 -> 0.00 mm, vias 1 -> 0
- net /CS_NRF24: track 44.5 -> 0.00 mm, vias 1 -> 0
- net +5V: track 41.7 -> 0.00 mm, vias 1 -> 0
- net /RESET: track 0.00 -> 36.8 mm
- net /CS_TOUCH: track 34.0 -> 0.00 mm, vias 1 -> 0
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Other:
- board size 76.2 x 73.7 mm -> 80 x 75 mm
- net class Default: trace_width 0.1524 -> 0.2
- board text removed: "Spectre-TX Multiprotocol Transmitter Proto V4"
- board text removed: "antoine@doussaud.org"

Commit message: v4 root
Parts:
- removed J6: GS2, Connectors:GS2
- removed R13, R14: 100K, Resistors_SMD:R_0805
- added REF**: Via, spectre:Via, F.Cu at (120.2, 59.6)
- added REF**: Via, spectre:Via, F.Cu at (118.2, 58.6)
- added REF**: Via, spectre:Via, F.Cu at (180.2, 48.6)
- added REF**: Via, spectre:Via, F.Cu at (179.2, 48.6)
- added REF**: Via, spectre:Via, F.Cu at (178.2, 48.6)
- added REF**: Via, spectre:Via, F.Cu at (177.2, 48.6)
- added REF**: Via, spectre:Via, F.Cu at (176.2, 48.6)
- added REF**: Via, spectre:Via, F.Cu at (155.7, 61.6)
- added REF**: Via, spectre:Via, F.Cu at (154.7, 61.6)
- added REF**: Via, spectre:Via, F.Cu at (153.7, 61.6)
- added REF**: Via, spectre:Via, F.Cu at (152.7, 61.6)
- added REF**: Via, spectre:Via, F.Cu at (151.7, 61.6)
- added REF**: Via, spectre:Via, F.Cu at (117.2, 58.6)
- added REF**: Via, spectre:Via, F.Cu at (150.7, 61.6)
- added REF**: Via, spectre:Via, F.Cu at (143.7, 85.6)
- added REF**: Via, spectre:Via, F.Cu at (142.7, 85.6)
- added REF**: Via, spectre:Via, F.Cu at (141.7, 85.6)
- added REF**: Via, spectre:Via, F.Cu at (140.7, 85.6)
- added REF**: Via, spectre:Via, F.Cu at (116.2, 58.6)
- added REF**: Via, spectre:Via, F.Cu at (115.2, 58.6)
- added REF**: Via, spectre:Via, F.Cu at (114.2, 58.6)
- added REF**: Via, spectre:Via, F.Cu at (120.2, 57.6)
- added REF**: Via, spectre:Via, F.Cu at (119.2, 57.6)
- added REF**: Via, spectre:Via, F.Cu at (118.2, 57.6)
- added REF**: Via, spectre:Via, F.Cu at (117.2, 57.6)
- added REF**: Via, spectre:Via, F.Cu at (116.2, 57.6)
- added REF**: Via, spectre:Via, F.Cu at (119.2, 59.6)
- added REF**: Via, spectre:Via, F.Cu at (115.2, 57.6)
- added REF**: Via, spectre:Via, F.Cu at (114.2, 57.6)
- added REF**: Via, spectre:Via, F.Cu at (120.2, 56.6)
- added REF**: Via, spectre:Via, F.Cu at (119.2, 56.6)
- added REF**: Via, spectre:Via, F.Cu at (118.2, 56.6)
- added REF**: Via, spectre:Via, F.Cu at (117.2, 56.6)
- added REF**: Via, spectre:Via, F.Cu at (116.2, 56.6)
- added REF**: Via, spectre:Via, F.Cu at (115.2, 56.6)
- added REF**: Via, spectre:Via, F.Cu at (114.2, 56.6)
- added REF**: Via, spectre:Via, F.Cu at (120.2, 55.6)
- added REF**: Via, spectre:Via, F.Cu at (118.2, 59.6)
- added REF**: Via, spectre:Via, F.Cu at (119.2, 55.6)
- added REF**: Via, spectre:Via, F.Cu at (118.2, 55.6)
- added REF**: Via, spectre:Via, F.Cu at (117.2, 55.6)
- added REF**: Via, spectre:Via, F.Cu at (116.2, 55.6)
- added REF**: Via, spectre:Via, F.Cu at (115.2, 55.6)
- added REF**: Via, spectre:Via, F.Cu at (114.2, 55.6)
- added REF**: Via, spectre:Via, F.Cu at (120.2, 54.6)
- added REF**: Via, spectre:Via, F.Cu at (119.2, 54.6)
- added REF**: Via, spectre:Via, F.Cu at (118.2, 54.6)
- added REF**: Via, spectre:Via, F.Cu at (117.2, 54.6)
- added REF**: Via, spectre:Via, F.Cu at (117.2, 59.6)
- added REF**: Via, spectre:Via, F.Cu at (116.2, 54.6)
- added REF**: Via, spectre:Via, F.Cu at (115.2, 54.6)
- added REF**: Via, spectre:Via, F.Cu at (114.2, 54.6)
- added REF**: Via, spectre:Via, F.Cu at (183.2, 51.6)
- added REF**: Via, spectre:Via, F.Cu at (182.2, 51.6)
- added REF**: Via, spectre:Via, F.Cu at (181.2, 51.6)
- added REF**: Via, spectre:Via, F.Cu at (180.2, 51.6)
- added REF**: Via, spectre:Via, F.Cu at (179.2, 51.6)
- added REF**: Via, spectre:Via, F.Cu at (178.2, 51.6)
- added REF**: Via, spectre:Via, F.Cu at (177.2, 51.6)
- added REF**: Via, spectre:Via, F.Cu at (116.2, 59.6)
- added REF**: Via, spectre:Via, F.Cu at (176.2, 51.6)
- added REF**: Via, spectre:Via, F.Cu at (155.7, 64.6)
- added REF**: Via, spectre:Via, F.Cu at (154.7, 64.6)
- added REF**: Via, spectre:Via, F.Cu at (153.7, 64.6)
- added REF**: Via, spectre:Via, F.Cu at (152.7, 64.6)
- added REF**: Via, spectre:Via, F.Cu at (151.7, 64.6)
- added REF**: Via, spectre:Via, F.Cu at (150.7, 64.6)
- added REF**: Via, spectre:Via, F.Cu at (143.7, 88.6)
- added REF**: Via, spectre:Via, F.Cu at (142.7, 88.6)
- added REF**: Via, spectre:Via, F.Cu at (141.7, 88.6)
- added REF**: Via, spectre:Via, F.Cu at (115.2, 59.6)
- added REF**: Via, spectre:Via, F.Cu at (140.7, 88.6)
- added REF**: Via, spectre:Via, F.Cu at (183.2, 50.6)
- added REF**: Via, spectre:Via, F.Cu at (182.2, 50.6)
- added REF**: Via, spectre:Via, F.Cu at (181.2, 50.6)
- added REF**: Via, spectre:Via, F.Cu at (180.2, 50.6)
- added REF**: Via, spectre:Via, F.Cu at (179.2, 50.6)
- added REF**: Via, spectre:Via, F.Cu at (178.2, 50.6)
- added REF**: Via, spectre:Via, F.Cu at (177.2, 50.6)
- added REF**: Via, spectre:Via, F.Cu at (176.2, 50.6)
- added REF**: Via, spectre:Via, F.Cu at (155.7, 63.6)
- added REF**: Via, spectre:Via, F.Cu at (114.2, 59.6)
- added REF**: Via, spectre:Via, F.Cu at (154.7, 63.6)
- added REF**: Via, spectre:Via, F.Cu at (153.7, 63.6)
- added REF**: Via, spectre:Via, F.Cu at (152.7, 63.6)
- added REF**: Via, spectre:Via, F.Cu at (151.7, 63.6)
- added REF**: Via, spectre:Via, F.Cu at (150.7, 63.6)
- added REF**: Via, spectre:Via, F.Cu at (143.7, 87.6)
- added REF**: Via, spectre:Via, F.Cu at (142.7, 87.6)
- added REF**: Via, spectre:Via, F.Cu at (141.7, 87.6)
- added REF**: Via, spectre:Via, F.Cu at (140.7, 87.6)
- added REF**: Via, spectre:Via, F.Cu at (183.2, 49.6)
- added REF**: Via, spectre:Via, F.Cu at (120.2, 58.6)
- added REF**: Via, spectre:Via, F.Cu at (182.2, 49.6)
- added REF**: Via, spectre:Via, F.Cu at (181.2, 49.6)
- added REF**: Via, spectre:Via, F.Cu at (180.2, 49.6)
- added REF**: Via, spectre:Via, F.Cu at (179.2, 49.6)
- added REF**: Via, spectre:Via, F.Cu at (178.2, 49.6)
- added REF**: Via, spectre:Via, F.Cu at (177.2, 49.6)
- added REF**: Via, spectre:Via, F.Cu at (176.2, 49.6)
- added REF**: Via, spectre:Via, F.Cu at (155.7, 62.6)
- added REF**: Via, spectre:Via, F.Cu at (154.7, 62.6)
- added REF**: Via, spectre:Via, F.Cu at (153.7, 62.6)
- added REF**: Via, spectre:Via, F.Cu at (119.2, 58.6)
- added REF**: Via, spectre:Via, F.Cu at (152.7, 62.6)
- added REF**: Via, spectre:Via, F.Cu at (151.7, 62.6)
- added REF**: Via, spectre:Via, F.Cu at (150.7, 62.6)
- added REF**: Via, spectre:Via, F.Cu at (143.7, 86.6)
- added REF**: Via, spectre:Via, F.Cu at (142.7, 86.6)
- added REF**: Via, spectre:Via, F.Cu at (141.7, 86.6)
- added REF**: Via, spectre:Via, F.Cu at (140.7, 86.6)
- added REF**: Via, spectre:Via, F.Cu at (183.2, 48.6)
- added REF**: Via, spectre:Via, F.Cu at (182.2, 48.6)
- added REF**: Via, spectre:Via, F.Cu at (181.2, 48.6)
- C11: value 0.1µF -> 0.1uF; moved to F.Cu
- C12: value 10µF -> 10uF; moved to F.Cu
- C6: value 1µF -> 1uF
- J7: moved to B.Cu
- R1: value 100k -> 100K
- U10: moved to F.Cu
- moved U10 112.1 mm to (158.7, 81.6), turned to 180 degrees
- moved R7 109.4 mm to (157.7, 92.1), turned to 270 degrees
- moved R9 107.2 mm to (127.7, 81.6)
- moved C7 101.7 mm to (127.7, 79.1), turned to 180 degrees
- moved C11 100.4 mm to (170.2, 73.6)
- moved C12 100.3 mm to (170.2, 76.1)
- moved C8 99.2 mm to (128.2, 73.1), turned to 270 degrees
- moved C9 95.6 mm to (127.7, 76.6), turned to 180 degrees
- moved C10 87.0 mm to (120.7, 73.1), turned to 270 degrees
- moved J7 84.6 mm to (184.2, 68.1)
- moved U7 80.6 mm to (123.2, 77.8), turned to 90 degrees
- moved L2 76.6 mm to (125.7, 73.1), turned to 270 degrees
- moved L1 70.3 mm to (123.2, 73.1), turned to 270 degrees
- moved LS1 57.9 mm to (123.7, 66.1), turned to 90 degrees
- moved C13 12.1 mm to (149.7, 95.6), turned to 0 degrees
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Connections:
- C7 pad 1: +5V -> +3V3
- C9 pad 1: +5V -> +3V3
- J2 pad 2: Net-(J2-Pad2) -> +3V3
- R9 pad 2: +5V -> +3V3
- U7 pad 7: +5V -> +3V3
- U7 pad 8: +5V -> +3V3
Routing:
- net +3V3: track 26.2 -> 306.1 mm, vias 0 -> 14
- net GND: track 13.4 -> 153.6 mm, vias 0 -> 22
- net /EXT_ADC_CH3: track 0.00 -> 104.2 mm
- net /MISO: track 0.00 -> 99.8 mm, vias 0 -> 8
- net /EXT_ADC_CH2: track 0.00 -> 93.0 mm
- net /MOSI: track 0.00 -> 92.6 mm, vias 0 -> 7
- net /SCK: track 0.00 -> 83.6 mm, vias 0 -> 6
- net /I2S_DATA: track 0.00 -> 82.8 mm, vias 0 -> 2
- net /I2S_BCLK: track 0.00 -> 67.8 mm, vias 0 -> 2
- net /NEOPIXEL: track 0.00 -> 66.8 mm, vias 0 -> 3
- net /EXT_ADC_CH0: track 0.00 -> 59.3 mm
- net /I2S_LRC: track 0.00 -> 55.0 mm, vias 0 -> 2
- net /CYRF_RST: track 0.00 -> 50.8 mm, vias 0 -> 6
- net /CS_ADC: track 0.00 -> 44.1 mm, vias 0 -> 2
- net /EXT_ADC_CH1: track 0.00 -> 41.9 mm
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
Commit message: rf tunning
Parts:
- added REF**: Via, spectre:Via, F.Cu at (148.4, 44.1)
- added REF**: Via, spectre:Via, F.Cu at (145.9, 44.1)
- added REF**: Via, spectre:Via, F.Cu at (148.4, 44.8)
- added REF**: Via, spectre:Via, F.Cu at (145.9, 44.8)
Changed lines of the file:
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@@
 (kicad_pcb (version 4) (host pcbnew 4.0.7-e2-6376~60~ubuntu17.10.1)
   (general
-    (links 314)
+    (links 318)
     (no_connects 0)
     (area 107.112999 39.012999 187.263001 114.163001)
@@
     (tracks 1065)
     (zones 0)
-    (modules 169)
+    (modules 173)
     (nets 102)
   )
@@
     (last_trace_width 0.2)
     (trace_clearance 0.1524)
-    (zone_clearance 0.508)
+    (zone_clearance 0.249281)
     (zone_45_only no)
     (trace_min 0.1524)
@@
     (aux_axis_origin 0 0)
     (grid_origin 107.188 69.088)
-    (visible_elements FFFFEF7F)
+    (visible_elements FFFFFF7F)
     (pcbplotparams
       (layerselection 0x010f0_80000001)
@@
   )
   (module spectre:Via (layer F.Cu)
+    (at 148.438 44.088)
+    (fp_text reference REF** (at 0 1.27) (layer F.SilkS) hide
+      (effects (font (size 1 1) (thickness 0.15)))
+    )
+    (fp_text value Via (at 0 -1.27) (layer F.Fab) hide
+      (effects (font (size 1 1) (thickness 0.15)))
+    )
+    (pad 1 thru_hole circle (at 0 0) (size 0.15 0.15) (drill 0.1) (layers *.Cu *.Mask)
+      (net 1 GND) (zone_connect 2))
+  )
+  (module spectre:Via (layer F.Cu)
+    (at 145.938 44.088)
+    (fp_text reference REF** (at 0 1.27) (layer F.SilkS) hide
+      (effects (font (size 1 1) (thickness 0.15)))
+    )
+    (fp_text value Via (at 0 -1.27) (layer F.Fab) hide
+      (effects (font (size 1 1) (thickness 0.15)))
+    )
+    (pad 1 thru_hole circle (at 0 0) (size 0.15 0.15) (drill 0.1) (layers *.Cu *.Mask)
+      (net 1 GND) (zone_connect 2))
+  )
+  (module spectre:Via (layer F.Cu)
+    (at 148.438 44.838)
+    (fp_text reference REF** (at 0 1.27) (layer F.SilkS) hide
+      (effects (font (size 1 1) (thickness 0.15)))
+    )
+    (fp_text value Via (at 0 -1.27) (layer F.Fab) hide
+      (effects (font (size 1 1) (thickness 0.15)))
+    )
+    (pad 1 thru_hole circle (at 0 0) (size 0.15 0.15) (drill 0.1) (layers *.Cu *.Mask)
+      (net 1 GND) (zone_connect 2))
+  )
+  (module spectre:Via (layer F.Cu)
+    (at 145.938 44.838)
+    (fp_text reference REF** (at 0 1.27) (layer F.SilkS) hide
+      (effects (font (size 1 1) (thickness 0.15)))
+    )
+    (fp_text value Via (at 0 -1.27) (layer F.Fab) hide
+      (effects (font (size 1 1) (thickness 0.15)))
+    )
+    (pad 1 thru_hole circle (at 0 0) (size 0.15 0.15) (drill 0.1) (layers *.Cu *.Mask)
+      (net 1 GND) (zone_connect 2))
+  )
+  (module spectre:Via (layer F.Cu)
     (at 120.188 59.588)
     (fp_text reference REF** (at 0 1.27) (layer F.SilkS) hide
@@
     (pad "" np_thru_hole oval (at -2.5 -0.8) (size 0.8 0.8) (drill 0.8) (layers *.Cu *.Mask))
     (pad "" np_thru_hole oval (at 2.5 -0.8) (size 0.8 0.8) (drill 0.8) (layers *.Cu *.Mask))
-    (model ${KISYS3DMOD}/Connectors_USB.3dshapes/USB_Micro-B_Wuerth-629105150521.wrl
-      (at (xyz 0 0 0))
+    (model /home/spectre/Downloads/Conn_USB-micro-2.0_socket_right-angle.wrl
+      (at (xyz 0 -0.05 0))
       (scale (xyz 1 1 1))
-      (rotate (xyz 0 0 0))
+      (rotate (xyz 0 0 -90))
     )
   )
@@
     (pad 1 smd rect (at -3.2 -2.7 270) (size 0.8 1.5) (layers F.Cu F.Paste F.Mask)
       (net 20 "Net-(J5-Pad1)"))
-    (model ${KISYS3DMOD}/Connectors.3dshapes/microSD_Card_Receptacle_Wuerth_693072010801.wrl
+    (model /home/spectre/Downloads/micro_sd_molex_wm6701.wrl
       (at (xyz 0 0 0))
       (scale (xyz 1 1 1))
@@
     (pad 39 smd rect (at 0.3 -2.45 90) (size 6 6) (layers F.Cu F.Paste F.Mask)
       (net 1 GND))
+    (model /home/spectre/dev/elec/kicad_projects/kicadlibs/kicad_lib_spectre/3d/KiCAD-ESP-WROOM-32.wrl
+      (at (xyz 0 0 0))
+      (scale (xyz 1 1 1))
+      (rotate (xyz 0 0 0))
+    )
   )
   (module RF_Modules:nRF24L01_Breakout (layer F.Cu)
@@
   (segment (start 127.095521 109.397365) (end 127.117709 109.460774) (width 0.2) (layer F.Cu) (net 101))
   (zone (net 1) (net_name GND) (layer F.Cu) (hatch edge 0.508)
-    (connect_pads (clearance 0.508))
+    (connect_pads (clearance 0.249281))
     (min_thickness 0.254)
     (fill yes (arc_segments 16) (thermal_gap 0.508) (thermal_bridge_width 0.508))
     (polygon
       (pts
-        (xy 107.188 114.088) (xy 106.188 39.088) (xy 187.188 39.088) (xy 187.188 114.088)
+        (xy 107.188 114.088) (xy 107.188 39.088) (xy 188.188 39.088) (xy 188.188 114.088)
       )
     )
   )
   (zone (net 1) (net_name GND) (layer B.Cu) (hatch edge 0.508)
-    (connect_pads (clearance 0.508))
+    (connect_pads (clearance 0.249281))
     (min_thickness 0.254)
     (fill yes (arc_segments 16) (thermal_gap 0.508) (thermal_bridge_width 0.508))
     (polygon
       (pts
-        (xy 107.188 114.088) (xy 106.188 39.088) (xy 187.188 39.088) (xy 187.188 114.088)
+        (xy 107.188 114.088) (xy 107.188 39.088) (xy 187.188 39.088) (xy 187.188 114.088)
       )
     )
