File: esp32_radio.kicad_pcb (KiCad board)
At the start: 2 copper layers, 80 x 75 mm, 74 parts, among them J1 RP-SMA, J2 LCD_TS, J4 USB_OTG, J5 Micro_SD_Card, J7 Conn_ADC, Q1 DMG3415U, Q2 Q_NPN_BCE, Q3 Q_NPN_BCE, Q4 Q_NPN_BCE, SW1 SW_Push, U1 RF4IN1, U10 MCP3008, U11 Joystick, U12 Joystick, U13 CC2500, U2 AP2112-3.3, U3 ESP32-WROOM, U4 nRF24L01, U5 MCP73831, U6 WS2812B, U7 MAX98357a, U8 CP2104, U9 XPT2046TS

Commit message: update
Parts:
- C11, C13, C16, C9: value 0.1uF -> 100nF
- D2: footprint LEDs:LED_0805 -> LED_SMD:LED_0603_1608Metric
- J4: footprint Connectors_USB:USB_Micro-B_Wuerth-629105150521_CircularHoles -> spectre:microUSB-smd-C40939
- J5: footprint Connectors:microSD_Card_Receptacle_Wuerth_693072010801 -> spectre:MicroSD_C125617
- SW1: footprint Buttons_Switches_SMD:SW_SPST_SKQG -> Button_Switch_THT:SW_PUSH_6mm
- moved J5 9.36 mm to (186.9, 83.8), turned to 90 degrees
- moved SW1 4.62 mm to (140.2, 112.1), turned to 180 degrees
- moved J4 1.78 mm to (117.3, 112.0)
Routing:
- net GND: track 81.4 -> 69.1 mm, vias 138 -> 141
- net /MISO: track 141.5 -> 131.0 mm, vias 5 -> 6
- net /RESET: track 56.9 -> 49.2 mm, vias 4 -> 1
- net +3V3: track 367.9 -> 375.2 mm
- net VBUS: track 31.4 -> 33.9 mm
- net /SCK: track 159.4 -> 161.2 mm
- net Net-(J5-Pad2): track 13.2 -> 11.8 mm
- net Net-(J5-Pad3): track 12.7 -> 11.4 mm
- net VBAT: track 67.8 -> 66.7 mm
- net Net-(J5-Pad5): track 9.91 -> 9.03 mm
- net /MOSI: track 150.3 -> 149.6 mm, vias 5 -> 6

Commit message: add 3d + fix mosfet
Parts:
- removed the J1 at (147.2, 41.6)
- added J1 (x3): RP-SMA, spectre:CON-SMA-EDGE, F.Cu at (147.2, 41.6)
Connections:
- Q1 pad 1: VBAT -> VBUS
- Q1 pad 2: VBUS -> Net-(C1-Pad1)
- Q1 pad 3: Net-(C1-Pad1) -> VBAT
Routing:
- net VBAT: track 66.7 -> 64.9 mm
- net Net-(C1-Pad1): track 12.4 -> 13.5 mm
- net VBUS: track 33.9 -> 34.7 mm

Commit message: update
Parts:
- removed C10: 220pF, Capacitor_SMD:C_0603_1608Metric
- removed C14: 10uF, Capacitor_SMD:C_0603_1608Metric
- removed C15: 1uF, Capacitor_SMD:C_0603_1608Metric
- removed the J1 at (147.2, 41.6) (x3)
- removed JP1: SolderJumper_3_Bridged12, Jumper:SolderJumper-3_P1.3mm_Bridged12_RoundedPad1.0x1.5mm
- removed L1, L2: Ferrite_Bead_Small, Resistors_SMD:R_0805
- removed LS1: Speaker, Pin_Headers:Pin_Header_Straight_1x02_Pitch2.54mm
- removed U8: CP2104, Housings_DFN_QFN:QFN-24-1EP_4x4mm_Pitch0.5mm
- added G***: LOGO, spectre:Logo, B.Cu at (149.5, 88.8)
- added G***: LOGO, spectre:bitmap, B.Cu at (147.1, 49.1)
- added J1: RP-SMA, spectre:CON-SMA-EDGE, F.Cu at (147.2, 41.6)
- added R22: 10K, Resistor_SMD:R_0603_1608Metric, F.Cu at (136.6, 21.9)
- added SW2: SW_Push, Button_Switch_THT:SW_Tactile_SPST_Angled_PTS645Vx58-2LFS, B.Cu at (158.9, 41.7)
- added SW3: SW_Push, Button_Switch_THT:SW_Tactile_SPST_Angled_PTS645Vx58-2LFS, B.Cu at (140.5, 41.8)
- added TP1: TestPoint, TestPoint:TestPoint_Pad_D1.0mm, F.Cu at (124.1, 106.3)
- added TP2: TestPoint, TestPoint:TestPoint_Pad_D1.0mm, F.Cu at (125.1, 107.7)
- added TP3: TestPoint, TestPoint:TestPoint_Pad_D1.0mm, B.Cu at (140.4, 101.4)
- added TP4: TestPoint, TestPoint:TestPoint_Pad_D1.0mm, B.Cu at (137.2, 102.8)
- added TP5: TestPoint, TestPoint:TestPoint_Pad_D1.0mm, F.Cu at (142.7, 135.1)
- added TP6: TestPoint, TestPoint:TestPoint_Pad_D1.0mm, F.Cu at (144.0, 130.0)
- added Y1: 12MHz, Crystal:Crystal_SMD_HC49-SD, F.Cu at (133.9, 104.1)
- BT1: footprint Connectors_JST:JST_PH_S2B-PH-K_02x2.00mm_Angled -> Connector_JST:JST_PH_B2B-PH-K_1x02_P2.00mm_Vertical
- C7: value 10uF -> 100nF
- C8: value 220pF -> 22pF
- C9: value 100nF -> 22pF
- J2: footprint spectre:TFT-2.4-IlI9341-18pin -> spectre:FPC_18
- R9: value 1M -> 10K
- SW1: value SW_Push -> SW_SPDT; footprint Button_Switch_THT:SW_PUSH_6mm -> Button_Switch_SMD:SW_SPDT_PCM12
- U7: value MAX98357a -> CH340G; footprint Housings_DFN_QFN:QFN-16-1EP_3x3mm_Pitch0.5mm -> Package_SO:SOIC-16_3.9x9.9mm_P1.27mm
- moved R9 67.5 mm to (157.4, 21.0)
- moved C9 64.9 mm to (109.7, 138.9)
- moved C8 64.7 mm to (109.7, 135.1), turned to 180 degrees
- moved C7 43.4 mm to (126.2, 122.4), turned to 90 degrees
- moved R13 31.4 mm to (165.7, 117.3)
- moved C4 27.1 mm to (128.8, 122.4)
- moved U7 18.5 mm to (130.0, 95.0), turned to 0 degrees
- moved J2 8.80 mm to (177.7, 100.1), turned to 90 degrees
- moved Q3 6.64 mm to (138.9, 93.2)
- moved Q2 6.00 mm to (138.9, 98.3)
- moved R4 5.11 mm to (135.6, 98.6), turned to 270 degrees
- moved BT1 4.60 mm to (129.9, 111.6), turned to 180 degrees
- moved J4 2.92 mm to (120.3, 112.0)
- moved R5 2.78 mm to (135.8, 93.2), turned to 270 degrees
- moved SW1 2.46 mm to (137.7, 112.0), turned to 0 degrees
Connections:
- C9 pad 1: +3V3 -> Net-(C9-Pad1)
- Q4 pad 1: /I2S_DATA -> /BUZZER
- R2 pad 2: Net-(R2-Pad2) -> /POWER
- R9 pad 1: Net-(R9-Pad1) -> +3V3
- R9 pad 2: +3V3 -> /B_L
- SW1 pad 1: GND -> Net-(SW1-Pad1)
- SW1 pad 2: /RESET -> /POWER
- U2 pad 3: Net-(R2-Pad2) -> /POWER
- U3 pad 10: /I2S_LRC -> /B_L
- U3 pad 11: /I2S_BCLK -> /B_R
- U3 pad 36: /IN+I2S_D -> /TS_IRQ
- U7 pad 1: /I2S_DATA -> GND
- U7 pad 11: GND -> Net-(U7-Pad11)
- U7 pad 13: Net-(U7-Pad13) -> /DTR
- U7 pad 14: /I2S_LRC -> /RTS
- U7 pad 15: GND -> Net-(U7-Pad15)
- U7 pad 16: /I2S_BCLK -> +3V3
- U7 pad 2: Net-(U7-Pad2) -> /RX0
- U7 pad 3: GND -> /TX0
- U7 pad 4: Net-(R9-Pad1) -> +3V3
- U7 pad 5: Net-(U7-Pad5) -> /D+
- U7 pad 6: Net-(U7-Pad6) -> /D-
- U7 pad 7: +3V3 -> Net-(C8-Pad1)
- U7 pad 8: +3V3 -> Net-(C9-Pad1)
Routing:
- net +3V3: track 375.2 -> 247.0 mm, vias 15 -> 8
- net /I2S_DATA: track 63.6 -> 0.00 mm, vias 2 -> 0
- net GND: track 69.1 -> 7.12 mm, vias 141 -> 84
- net /MOSI: track 149.6 -> 88.8 mm, vias 6 -> 3
- net /SCK: track 161.2 -> 101.6 mm, vias 5 -> 2
- net /MISO: track 131.0 -> 75.6 mm, vias 6 -> 2
- net /I2S_LRC: track 49.3 -> 0.00 mm, vias 4 -> 0
- net /I2S_BCLK: track 48.1 -> 0.00 mm, vias 4 -> 0
- net /B_L: track 0.00 -> 42.1 mm, vias 0 -> 3
- net /B_R: track 0.00 -> 40.5 mm, vias 0 -> 4
- net /RESET: track 49.2 -> 20.9 mm, vias 1 -> 0
- net /CS_SD: track 47.0 -> 23.1 mm, vias 2 -> 1
- net /INT_ADC_CH0: track 58.9 -> 36.3 mm
- net /D-: track 22.2 -> 0.00 mm, vias 2 -> 0
- net /D+: track 21.3 -> 0.00 mm, vias 2 -> 0
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Other:
- board text added: "Spectre-Tx Multiprocol Transmitter Proto V6"
- board text removed: "Spectre-Tx Multiprocol Transmitter Proto V5"

Commit message: v6
Parts:
- removed Q3: Q_NPN_BCE, TO_SOT_Packages_SMD:SOT-23
- removed the R14 at (167.1, 88.4)
- removed the R4 at (135.6, 98.6)
- removed R6: 4.7K, Resistor_SMD:R_0603_1608Metric
- removed TP1, TP2, TP3, TP4, TP5, TP6: TestPoint, TestPoint:TestPoint_Pad_D1.0mm
- removed U13: CC2500, Pin_Headers:Pin_Header_Straight_2x06_Pitch2.54mm
- removed U7: CH340G, Package_SO:SOIC-16_3.9x9.9mm_P1.27mm
- added R9: 100K, Resistor_SMD:R_0603_1608Metric, F.Cu at (164.7, 94.6)
- BT1: value Battery_Cell -> 1S Battery
- Q2: value Q_NPN_BCE -> UMH3N; footprint TO_SOT_Packages_SMD:SOT-23 -> Package_TO_SOT_SMD:SOT-363_SC-70-6
- R13: renamed from R18; moved to B.Cu
- R14: renamed from R19; moved to B.Cu
- R15: renamed from R20; moved to B.Cu
- R16: renamed from R21; moved to B.Cu
- R5: value 10K -> 4.7K
- U1: renamed from U3; footprint spectre:ESP32-WROOM-WROVER -> spectre:ESP32-WROOM-32
- U4: value nRF24L01 -> CH340G; footprint spectre:nRF24L01_Breakout -> Package_SO:SOIC-16_3.9x9.9mm_P1.27mm
- Y1: footprint Crystal:Crystal_SMD_HC49-SD -> Crystal:Crystal_SMD_3225-4Pin_3.2x2.5mm
- moved C9 55.3 mm to (137.4, 91.1), turned to 0 degrees
- moved C8 46.7 mm to (137.4, 97.6)
- moved R21 27.5 mm to (167.1, 46.7), turned to 180 degrees
- moved R22 27.5 mm to (129.2, 48.4), turned to 90 degrees
- moved Q4 26.9 mm to (128.7, 91.6)
- moved U4 23.4 mm to (130.7, 99.6), turned to 180 degrees
- moved C13 22.2 mm to (184.7, 80.6), turned to 270 degrees
- moved C14 20.6 mm to (182.7, 80.6), turned to 270 degrees
- moved C6 18.8 mm to (125.9, 103.8), turned to 270 degrees
- moved C7 18.7 mm to (124.2, 103.8), turned to 270 degrees
- moved R13 18.5 mm to (150.7, 69.1)
- moved R14 18.3 mm to (148.7, 69.1)
- moved R15 18.0 mm to (146.7, 69.1)
- moved R16 17.8 mm to (144.7, 69.1)
- moved J2 16.3 mm to (167.2, 87.6), turned to 270 degrees
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- renumbered C18 to C1, C13 to C10, C16 to C11, C17 to C12, C11 to C13, C12 to C14, C6 to C15, C1 to C2, C2 to C3, C3 to C4, C4 to C6, J4 to J1, J1 to J3, J5 to J4, J7 to J5, R15 to R10, R16 to R11, R17 to R12, R10 to R17, R11 to R18, R12 to R19, R8 to R20, R9 to R21, R13 to R4, R7 to R8, SW2 to SW1, SW3 to SW2, SW1 to SW3, U11 to U10, U12 to U11, U6 to U12, U5 to U3, U9 to U5, U10 to U6, U1 to U8
Connections:
- Q2 pad 1: Net-(Q2-Pad1) -> /RTS
- Q2 pad 2: /GPIO_0 -> /DTR
- Q2 pad 3: /DTR -> /GPIO_0
- Q4 pad 1: /BUZZER -> /GPIO_0
- R5 pad 1: Net-(Q3-Pad1) -> GND
- R5 pad 2: /DTR -> Net-(R5-Pad2)
- U1 pad 10: /B_L -> /CS_SD
- U1 pad 11: /B_R -> /CS_LCD
- U1 pad 12: /CS_CC25 -> /LCD_CMD
- U1 pad 13: /CS_A7105 -> /SCK
- U1 pad 14: /PE2 -> /MISO
- U1 pad 16: /PE1 -> /MOSI
- U1 pad 23: /CS_LCD -> /CS_CYRF
- U1 pad 24: /LCD_CMD -> /CS_NRF24
- U1 pad 26: /CS_TOUCH -> /CS_CC25
- U1 pad 27: /CS_SD -> /CS_A7105
- U1 pad 30: /SCK -> /PE2
- U1 pad 31: /MISO -> /PE1
- U1 pad 36: /TS_IRQ -> /B_R
- U1 pad 37: /MOSI -> /B_L
- U1 pad 8: /CS_CYRF -> /TS_IRQ
- U1 pad 9: /CS_NRF24 -> /CS_TOUCH
- U10 pad 2: /INT_ADC_CH1 -> /INT_ADC_CH3
- U10 pad 5: /INT_ADC_CH0 -> /INT_ADC_CH2
- U11 pad 2: /INT_ADC_CH3 -> /INT_ADC_CH0
- U11 pad 5: /INT_ADC_CH2 -> /INT_ADC_CH1
- U3 pad 5: Net-(R6-Pad2) -> Net-(R5-Pad2)
- U4 pad 2: +3V3 -> /RX0
- U4 pad 3: +3V3 -> /TX0
- U4 pad 4: /CS_NRF24 -> +3V3
- U4 pad 5: /SCK -> /D+
- U4 pad 6: /MOSI -> /D-
- U4 pad 7: /MISO -> Net-(C8-Pad1)
- U4 pad 8: Net-(U4-Pad8) -> Net-(C9-Pad1)
- Y1 pad 2: Net-(C9-Pad1) -> GND
Routing:
- net +3V3: track 247.0 -> 317.7 mm, vias 8 -> 7
- net /INT_ADC_CH0: track 36.3 -> 83.5 mm
- net /INT_ADC_CH1: track 28.0 -> 69.4 mm, vias 2 -> 1
- net /B_L: track 42.1 -> 83.3 mm, vias 3 -> 2
- net /B_R: track 40.5 -> 73.5 mm
- net /INT_ADC_CH3: track 76.5 -> 46.1 mm, vias 3 -> 1
- net /MISO: track 75.6 -> 104.8 mm, vias 2 -> 6
- net /GPIO_0: track 0.00 -> 28.0 mm, vias 0 -> 2
- net /POWER: track 2.15 -> 26.1 mm, vias 0 -> 2
- net /D-: track 0.00 -> 21.9 mm
- net /D+: track 0.00 -> 20.8 mm
- net /CYRF_RST: track 43.3 -> 28.1 mm
- net /CS_LCD: track 21.4 -> 8.81 mm, vias 0 -> 1
- net /BUZZER: track 12.1 -> 0.00 mm
- net Net-(J4-Pad2): track 0.00 -> 12.0 mm, vias 0 -> 2
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